Commit message: Add files via upload

File: p_mrivadeneira/p_mrivadeneira_description/urdf/p_mrivadeneira.gazebo.xacro (robot description, xacro)
@@ -4,6 +4,6 @@
   <xacro:arg name="camera_visual" default="false"/>
   <xacro:arg name="imu_visual"    default="false"/>
+  <!-- +++++++++++++++++++++++++++++++++++++++ Including URDF references +++++++++++++++++++++++++++++++++++++++ -->
   <gazebo reference="base_link">
-<!--    <material>Gazebo/DarkGrey</material>-->
     <material>Gazebo/${player_color}</material>
   </gazebo>
@@ -12,14 +12,14 @@
   </gazebo>
   <gazebo reference="left_arm">
-    <material>Gazebo/${player_color}</material>
+      <material>Gazebo/Gray</material>
   </gazebo>
     <gazebo reference="left_arm_base">
-    <material>Gazebo/${player_color}</material>
+      <material>Gazebo/Gray</material>
   </gazebo>
     <gazebo reference="right_arm">
-    <material>Gazebo/${player_color}</material>
+      <material>Gazebo/Gray</material>
   </gazebo>
     <gazebo reference="right_arm_base">
-    <material>Gazebo/${player_color}</material>
+      <material>Gazebo/Gray</material>
   </gazebo>
   <gazebo reference="wheel_left_link">

File: p_mrivadeneira/p_mrivadeneira_description/urdf/p_mrivadeneira.urdf.xacro (robot description, xacro)
@@ -13,4 +13,5 @@
 <!--  <xacro:include filename="$(find turtlebot3_description)/urdf/turtlebot3_waffle_pi.gazebo.xacro"/>-->
   <xacro:include filename="$(find p_mrivadeneira_description)/urdf/p_mrivadeneira.gazebo.xacro"/>
+<!-- +++++++++++++++++++++++++++++++++++++++ BASIC TURTLEBOT +++++++++++++++++++++++++++++++++++++++ -->
 <!--  Define links and joints-->
   <link name="base_footprint"/>
@@ -55,6 +56,5 @@
         <mesh filename="package://turtlebot3_description/meshes/wheels/left_tire.stl" scale="0.001 0.001 0.001"/>
       </geometry>
-<!--      <material name="dark"/>-->
-      <material name="$(arg player_color)"/>
+      <material name="dark"/>
      </visual>
     <collision>
@@ -84,6 +84,5 @@
         <mesh filename="package://turtlebot3_description/meshes/wheels/right_tire.stl" scale="0.001 0.001 0.001"/>
       </geometry>
-<!--      <material name="dark"/>-->
-      <material name="$(arg player_color)"/>
+      <material name="dark"/>
     </visual>
     <collision>
@@ -199,4 +198,5 @@
   </joint>
   <link name="camera_rgb_optical_frame"/>
+  <!-- +++++++++++++++++++++++++++++++++++++++ EXTRAS FOR TURTLEBOT +++++++++++++++++++++++++++++++++++++++ -->
     <!--base_link to antenna-->
   <link name="antenna">
@@ -206,4 +206,5 @@
         <cylinder length="0.15" radius="0.005"/>
       </geometry>
+      <material name="$(arg player_color)"/>
     </visual>
   </link>
@@ -213,71 +214,158 @@
     <child link="antenna"/>
   </joint>
-<!--  &lt;!&ndash;Left arm&ndash;&gt;-->
-<!--  <link name="left_arm_base">-->
-<!--    <visual>-->
-<!--      <origin rpy="0 0 0" xyz="0 0 0"/>-->
-<!--      <geometry>-->
-<!--        <cylinder length="0.05" radius="0.02"/>-->
-<!--      </geometry>-->
-<!--    </visual>-->
-<!--  </link>-->
-<!--  <joint name="base_link_to_left_arm_base" type="fixed">-->
-<!--    <origin rpy="0 0 0" xyz="0.04 -0.095 0.11"/>-->
-<!--    <parent link="base_link"/>-->
-<!--    <child link="left_arm_base"/>-->
-<!--  </joint>-->
-<!--    <link name="left_arm">-->
-<!--    <visual>-->
-<!--      <origin xyz="0 -0.1 0" rpy="0 0 0"/>-->
-<!--      <geometry>-->
-<!--        <box size="0.04 0.2 0.050"/>-->
-<!--      </geometry>-->
-<!--    </visual>-->
-<!--  </link>-->
-<!--  <joint name="left_arm_base_to_left_arm" type="fixed">-->
-<!--    <origin rpy="0 0 0" xyz="0 0 0"/>-->
-<!--    <parent link="left_arm_base"/>-->
-<!--    <child link="left_arm"/>-->
-<!--  </joint>-->
-<!--  &lt;!&ndash;  <joint name="left_arm_base_to_left_arm" type="revolute">&ndash;&gt;-->
-<!--&lt;!&ndash;    <axis xyz="0 0 1"/>&ndash;&gt;-->
-<!--&lt;!&ndash;    <limit effort="1000.0" lower="0.0" upper="1.57" velocity="0.5"/>&ndash;&gt;-->
-<!--&lt;!&ndash;    <origin rpy="0 0 0" xyz="0 0 1"/>&ndash;&gt;-->
-<!--&lt;!&ndash;    <parent link="left_arm_base"/>&ndash;&gt;-->
-<!--&lt;!&ndash;    <child link="left_arm"/>&ndash;&gt;-->
-<!--&lt;!&ndash;  </joint>&ndash;&gt;-->
-<!--&lt;!&ndash;Right arm&ndash;&gt;-->
-<!--  <link name="right_arm_base">-->
-<!--    <visual>-->
-<!--      <origin rpy="0 0 0" xyz="0 0 0"/>-->
-<!--      <geometry>-->
-<!--        <cylinder length="0.05" radius="0.02"/>-->
-<!--      </geometry>-->
-<!--    </visual>-->
-<!--  </link>-->
-<!--  <joint name="base_link_to_right_arm_base" type="fixed">-->
-<!--    <origin rpy="0 0 0" xyz="0.04 0.095 0.11"/>-->
-<!--    <parent link="base_link"/>-->
-<!--    <child link="right_arm_base"/>-->
-<!--  </joint>-->
-<!--    <link name="right_arm">-->
-<!--    <visual>-->
-<!--      <origin xyz="0 0.1 0" rpy="0 0 0"/>-->
-<!--      <geometry>-->
-<!--        <box size="0.04 0.2 0.050"/>-->
-<!--      </geometry>-->
-<!--    </visual>-->
-<!--  </link>-->
-<!--  <joint name="left_arm_base_to_right_arm" type="fixed">-->
-<!--    <origin rpy="0 0 0" xyz="0 0 0"/>-->
-<!--    <parent link="right_arm_base"/>-->
-<!--    <child link="right_arm"/>-->
-<!--  </joint>-->
-<!--  &lt;!&ndash;  <joint name="left_arm_base_to_left_arm" type="revolute">&ndash;&gt;-->
-<!--&lt;!&ndash;    <axis xyz="0 0 1"/>&ndash;&gt;-->
-<!--&lt;!&ndash;    <limit effort="1000.0" lower="0.0" upper="1.57" velocity="0.5"/>&ndash;&gt;-->
-<!--&lt;!&ndash;    <origin rpy="0 0 0" xyz="0 0 1"/>&ndash;&gt;-->
-<!--&lt;!&ndash;    <parent link="left_arm_base"/>&ndash;&gt;-->
-<!--&lt;!&ndash;    <child link="left_arm"/>&ndash;&gt;-->
-<!--&lt;!&ndash;  </joint>&ndash;&gt;-->
+  <!--Right arm-->
+  <link name="right_arm_base">
+    <visual>
+      <origin rpy="0 0 0" xyz="0 0 0"/>
+      <geometry>
+        <cylinder length="0.015" radius="0.02"/>
+      </geometry>
+      <material name="dark"/>
+    </visual>
+    <collision>
+      <origin rpy="0 0 0" xyz="0 0 0"/>
+      <geometry>
+        <cylinder length="0.015" radius="0.02"/>
+      </geometry>
+    </collision>
+    <inertial>
+      <origin rpy="0 0 0" xyz="0 0 0"/>
+      <mass value="0.005"/>
+      <inertia
+        ixx="0.001" ixy="0.0" ixz="0.0"
+        iyy="0.001" iyz="0.0"
+        izz="0.001"
+      />
+    </inertial>
+  </link>
+  <joint name="base_link_to_right_arm_base" type="fixed">
+    <origin rpy="0 0 0" xyz="0.04 -0.095 0.0985"/>
+    <parent link="base_link"/>
+    <child link="right_arm_base"/>
+  </joint>
+    <link name="right_arm">
+    <visual>
+      <origin xyz="-0.1 0 0" rpy="0 0 0"/>
+      <geometry>
+        <box size="0.2 0.04 0.0150"/>
+      </geometry>
+      <material name="dark"/>
+    </visual>
+    <collision>
+      <origin xyz="-0.1 0 0" rpy="0 0 0"/>
+      <geometry>
+        <box size="0.2 0.04 0.0150"/>
+      </geometry>
+    </collision>
+    <inertial>
+      <origin rpy="0 0 0" xyz="0 0 0"/>
+      <mass value="0.005"/>
+      <inertia
+        ixx="0.001" ixy="0.0" ixz="0.0"
+        iyy="0.001" iyz="0.0"
+        izz="0.001"
+      />
+    </inertial>
+  </link>
+  <joint name="right_arm_base_to_right_arm" type="revolute">
+    <axis xyz="0 0 1"/>
+    <limit effort="1000.0" lower="0.0" upper="1.8" velocity="0.2"/>
+    <origin rpy="0 0 0" xyz="0 0 0"/>
+    <parent link="right_arm_base"/>
+    <child link="right_arm"/>
+    <dynamics damping="0.7" />
+  </joint>
+   <!--Left arm-->
+  <link name="left_arm_base">
+    <visual>
+      <origin rpy="0 0 0" xyz="0 0 0"/>
+      <geometry>
+        <cylinder length="0.015" radius="0.02"/>
+      </geometry>
+      <material name="dark"/>
+    </visual>
+    <collision>
+      <origin rpy="0 0 0" xyz="0 0 0"/>
+      <geometry>
+        <cylinder length="0.015" radius="0.02"/>
+      </geometry>
+    </collision>
+    <inertial>
+      <origin rpy="0 0 0" xyz="0 0 0"/>
+      <mass value="0.005"/>
+      <inertia
+        ixx="0.001" ixy="0.0" ixz="0.0"
+        iyy="0.001" iyz="0.0"
+        izz="0.001"
+      />
+    </inertial>
+  </link>
+  <joint name="base_link_to_left_arm_base" type="fixed">
+    <origin rpy="0 0 0" xyz="0.04 0.095 0.0985"/>
+    <parent link="base_link"/>
+    <child link="left_arm_base"/>
+  </joint>
+    <link name="left_arm">
+    <visual>
+      <origin xyz="-0.1 0 0" rpy="0 0 0"/>
+      <geometry>
+        <box size="0.2 0.04 0.0150"/>
+      </geometry>
+      <material name="dark"/>
+    </visual>
+    <collision>
+      <origin xyz="-0.1 0 0" rpy="0 0 0"/>
+      <geometry>
+        <box size="0.2 0.04 0.0150"/>
+      </geometry>
+    </collision>
+    <inertial>
+      <origin rpy="0 0 0" xyz="0 0 0"/>
+      <mass value="0.005"/>
+      <inertia
+        ixx="0.001" ixy="0.0" ixz="0.0"
+        iyy="0.001" iyz="0.0"
+        izz="0.001"
+      />
+    </inertial>
+  </link>
+    <joint name="left_arm_base_to_left_arm" type="revolute">
+    <axis xyz="0 0 1"/>
+    <limit effort="1000.0" lower="-1.8" upper="0.0" velocity="0.2"/>
+    <origin rpy="0 0 0" xyz="0 0 0"/>
+    <parent link="left_arm_base"/>
+    <child link="left_arm"/>
+    <dynamics damping="0.7" />
+  </joint>
+<!-- +++++++++++++++++++++++++++++++++++++++ Gazebo Related Part ++++++++++++++++++++++++++++++++++++++++++++ -->
+<!--  ROS control plug-in for Gazebo-->
+  <gazebo>
+    <plugin name="gazebo_ros_control" filename="libgazebo_ros_control.so">
+        <robotNamespace>/${player_name}</robotNamespace>
+        <robotSimType>gazebo_ros_control/DefaultRobotHWSim</robotSimType>
+        <robotParam>/${player_name}/robot_description</robotParam>
+        <legacyModeNS>true</legacyModeNS>
+    </plugin>
+  </gazebo>
+<!--  Transmission definition for arms-->
+  <transmission name="right_arm_base_to_right_arm_transmission">
+    <type>transmission_interface/SimpleTransmission</type>
+    <joint name="right_arm_base_to_right_arm">
+      <hardwareInterface>hardware_interface/EffortJointInterface</hardwareInterface>
+    </joint>
+    <actuator name="motor1">
+      <hardwareInterface>hardware_interface/EffortJointInterface</hardwareInterface>
+      <mechanicalReduction>1</mechanicalReduction>
+    </actuator>
+  </transmission>
+    <transmission name="left_arm_base_to_left_arm_transmission">
+    <type>transmission_interface/SimpleTransmission</type>
+    <joint name="left_arm_base_to_left_arm">
+      <hardwareInterface>hardware_interface/EffortJointInterface</hardwareInterface>
+    </joint>
+    <actuator name="motor2">
+      <hardwareInterface>hardware_interface/EffortJointInterface</hardwareInterface>
+      <mechanicalReduction>1</mechanicalReduction>
+    </actuator>
+  </transmission>
 </robot>
