Commit message: Driver improvements

File: Trabalho3-Grupo1/p_mrivadeneira/p_mrivadeneira_description/urdf/p_mrivadeneira.gazebo.xacro (robot description, xacro)
@@ -8,7 +8,7 @@
     <material>Gazebo/${player_color}</material>
   </gazebo>
-  <gazebo reference="antenna">
-    <material>Gazebo/${player_color}</material>
-  </gazebo>
+<!--  <gazebo reference="antenna">-->
+<!--    <material>Gazebo/${player_color}</material>-->
+<!--  </gazebo>-->
   <gazebo reference="left_arm">
       <material>Gazebo/Gray</material>

File: Trabalho3-Grupo1/p_mrivadeneira/p_mrivadeneira_description/urdf/p_mrivadeneira.urdf.xacro (robot description, xacro)
@@ -200,18 +200,18 @@
 <!--  &lt;!&ndash; +++++++++++++++++++++++++++++++++++++++ EXTRAS FOR TURTLEBOT +++++++++++++++++++++++++++++++++++++++ &ndash;&gt;-->
     <!--base_link to antenna-->
-  <link name="antenna">
-    <visual>
-      <origin rpy="0 0 0" xyz="0 0 0"/>
-      <geometry>
-        <cylinder length="0.15" radius="0.005"/>
-      </geometry>
-      <material name="$(arg player_color)"/>
-    </visual>
-  </link>
-  <joint name="base_link_to_antenna" type="fixed">
-    <origin rpy="0 0 0" xyz="0.05 0 0.16"/>
-    <parent link="base_link"/>
-    <child link="antenna"/>
-  </joint>
+<!--  <link name="antenna">-->
+<!--    <visual>-->
+<!--      <origin rpy="0 0 0" xyz="0 0 0"/>-->
+<!--      <geometry>-->
+<!--        <cylinder length="0.15" radius="0.005"/>-->
+<!--      </geometry>-->
+<!--      <material name="$(arg player_color)"/>-->
+<!--    </visual>-->
+<!--  </link>-->
+<!--  <joint name="base_link_to_antenna" type="fixed">-->
+<!--    <origin rpy="0 0 0" xyz="0.05 0 0.16"/>-->
+<!--    <parent link="base_link"/>-->
+<!--    <child link="antenna"/>-->
+<!--  </joint>-->
   <!--Right arm-->
   <link name="right_arm_base">
